Commit message: Update 3d box insertion

File: assets/urdf/Box3D/box3D.urdf (robot description, URDF)
Before this commit: robot box3d_insertion, 12 links, 11 joints
Links:
- removed link box
- removed link dummy
- removed link dummy2
- removed link dummy3
- removed link dummy4
- removed link dummy5
- link part1: geometry collision box size=2. 0.8725 0.2; visual box size=2. 0.8725 0.2
- link part2: geometry collision box size=2. 0.8725 0.2; visual box size=2. 0.8725 0.2
- link part3: geometry collision box size=0.8725 2. 0.2; visual box size=0.8725 2. 0.2
- link part4: geometry collision box size=0.8725 2. 0.2; visual box size=0.8725 2. 0.2
Joints:
- removed joint p_joint_x
- removed joint p_joint_y
- removed joint p_joint_z
- removed joint r_joint_x
- removed joint r_joint_y
- removed joint r_joint_z
- joint base_to_part1: origin xyz=0 -0.1775 0 -> xyz=0 -0.56375 0
- joint base_to_part2: origin xyz=0 0.1775 0 -> xyz=0 0.56375 0
- joint base_to_part3: origin xyz=0.1775 0. 0 -> xyz=0.56375 0. 0
- joint base_to_part4: origin xyz=-0.1775 0. 0 -> xyz=-0.56375 0. 0

File: assets/urdf/Box3D/peg.urdf (robot description, URDF)
Before this commit: robot box3d_insertion, 12 links, 11 joints
Links:
- removed link box
- removed link part1
- removed link part2
- removed link part3
- removed link part4
- removed link table
- added link ee, mass 1.; collision box size=0.25 0.25 0.25; visual box size=0.25 0.25 0.25
Joints:
- removed joint base_to_part1
- removed joint base_to_part2
- removed joint base_to_part3
- removed joint base_to_part4
- removed joint base_to_table
- joint r_joint_z: child box -> ee
